Commit message: fix: relative paths instead of using 'package://'

File: astro_max.urdf (robot description, URDF)
Before this commit: robot astro_max, 5 links, 4 joints
Links:
- link body_frd: geometry collision mesh filename=meshes/collision/body_frd.STL; visual mesh filename=meshes/visual/body_frd.STL
- link rotor_1_ccw: geometry collision mesh filename=meshes/collision/rotor_ccw.STL; visual mesh filename=meshes/visual/prop_bolts_ccw.STL
- link rotor_2_cw: geometry collision mesh filename=meshes/collision/rotor_cw.STL; visual mesh filename=meshes/visual/prop_bolts_cw.STL
- link rotor_3_ccw: geometry collision mesh filename=meshes/collision/rotor_ccw.STL; visual mesh filename=meshes/visual/prop_bolts_ccw.STL
- link rotor_4_cw: geometry collision mesh filename=meshes/collision/rotor_cw.STL; visual mesh filename=meshes/visual/prop_bolts_cw.STL

Commit message: fix: unstable sim due to offset rotor COMs and small masses
Note values are still not accurate. For now, chosen to match the quad_x values that fly well

File: astro_max.urdf (robot description, URDF)
Before this commit: robot astro_max, 5 links, 4 joints
Links:
- link body_frd: mass 0.88897 -> 8.18
- link rotor_1_ccw: mass 0.097019 -> 0.25
- link rotor_2_cw: mass 0.098646 -> 0.25
- link rotor_3_ccw: mass 0.098645 -> 0.25
- link rotor_4_cw: mass 0.098646 -> 0.25
